Commit message: Add urdf

File: Project4/catkin_ws/src/panda_pkg/urdf/panda_arm_hand.urdf.xacro (robot description, xacro)
@@ -5,11 +5,10 @@
 <!-- =================================================================================== -->
 <robot name="panda">
-<!-- <link name="dummy_link">
-  </link>
-  <joint name="dummy_joint" type="fixed">
-    <origin rpy="0 0 0" xyz="0 0 0"/>
-    <parent link="dummy_link"/>
+<link name="world" />
+  <joint name="fixed" type="fixed">
+    <!-- <origin rpy="0 0 0" xyz="0 0 0"/> -->
+    <parent link="world"/>
     <child link="panda_link0"/>
-  </joint> -->
+  </joint>
     <link name="panda_link0">
         <visual>
@@ -405,4 +404,18 @@
             </geometry>
         </visual>
+        <collision>
+      <origin xyz="0 0 0" rpy="0 0 0" />
+      <geometry>
+        <cylinder length="${0.0}" radius="${0.0}" />
+      </geometry>
+    </collision>
+        <inertial>
+        <origin xyz="0 0 0" rpy="0 0 0" />
+        <mass value="1" />
+        <inertia
+          ixx="0.0" ixy="0.0" ixz="0.0"
+          iyy="0.0" iyz="0.0"
+          izz="0.0" />
+    </inertial>
     </link>
     <link name="panda_rightfinger">
@@ -413,4 +426,18 @@
             </geometry>
         </visual>
+<collision>
+      <origin xyz="0 0 0" rpy="0 0 0" />
+      <geometry>
+        <cylinder length="${0.0}" radius="${0.0}" />
+      </geometry>
+    </collision>
+ <inertial>
+        <origin xyz="0 0 0" rpy="0 0 0" />
+        <mass value="1" />
+        <inertia
+          ixx="0.0" ixy="0.0" ixz="0.0"
+          iyy="0.0" iyz="0.0"
+          izz="0.0" />
+    </inertial>
     </link>
     <joint name="panda_finger_joint1" type="prismatic">
